File: hardware/cards/alu/kicad/v3.2/alu-v3.2-sheet4.kicad_sch (KiCad schematic)
At the start: 10 parts, among them IC14 74*86, IC15 74*86, IC16 74*244, IC17 74*244, IC18 74*08, IC19 74*08, IC20 74*244, IC21 74*32, IC22 74*32, IC23 74*244

Commit message: fix(kicad): readable converted schematics - overlaps 42,847 -> 3,147, nothing off the frame; CF sheet 0 overlaps
- tools/kicad/sch_overlaps.py: calibrated readability check (text/text, text/body, text/line, off frame/title block)
- eagle_sch_to_kicad.py: fields placed from Eagle's smashed attributes or the symbol's >NAME/>VALUE with Eagle's align,
  size and ratio, readable angles; fields Eagle never shows hidden (FABC96R shows only its pin name); pin numbers hidden
  where every Eagle pin hides them; Eagle-hidden layers dropped (the stray SpiceOrder text); labels on their own wires,
  converter labels only where KiCad needs them; rotate-then-mirror fixed for MR90/MR270 in pin_world/no-connects;
  each sheet on the smallest page that holds it, centred clear of the title block
- finish_board.py: stable footprint-library choice (DRC counts no longer vary run to run)
- all 37 projects regenerated: netlist proofs unchanged (34 MATCH, 2 schematic-only, video Fusion export MISMATCH as
  before); DRC same or better; ERC up (loose wire ends onto graphic buses no longer hidden by labels; explained per README)
- CF card: gate names off the gate bodies, U3 clear of its title, 5.08 mm connector pins; rebuilt: DRC 0/0, proof MATCH
- schematic PDFs regenerated (tools/sch_to_pdf.py, 37/37)

Co-Authored-By: Claude Opus 5.5 <noreply@anthropic.com>
Connections:
- net N$100: no longer names the net of IC15.6 (O), IC17.15 (A3)
- net N$101: no longer names the net of IC15.8 (O), IC17.17 (A4)
- net N$77: no longer names the net of IC21.3 (O), IC23.2 (A1)
- net N$78: no longer names the net of IC21.6 (O), IC23.4 (A2)
- net N$79: no longer names the net of IC21.8 (O), IC23.6 (A3)
- net N$81: no longer names the net of IC21.11 (O), IC23.8 (A4)
- net N$82: no longer names the net of IC22.3 (O), IC23.11 (A1)
- net N$83: no longer names the net of IC22.6 (O), IC23.13 (A2)
- net N$84: no longer names the net of IC22.8 (O), IC23.15 (A3)
- net N$85: no longer names the net of IC22.11 (O), IC23.17 (A4)
- net N$86: no longer names the net of IC18.3 (O), IC20.2 (A1)
- net N$87: no longer names the net of IC18.6 (O), IC20.4 (A2)
- net N$88: no longer names the net of IC18.8 (O), IC20.6 (A3)
- net N$89: no longer names the net of IC18.11 (O), IC20.8 (A4)
- net N$90: no longer names the net of IC19.11 (O), IC20.11 (A1)
- net N$91: no longer names the net of IC19.3 (O), IC20.13 (A2)
- net N$92: no longer names the net of IC19.6 (O), IC20.15 (A3)
- net N$93: no longer names the net of IC19.8 (O), IC20.17 (A4)
- net N$94: no longer names the net of IC14.3 (O), IC17.2 (A1)
- net N$95: no longer names the net of IC14.6 (O), IC17.4 (A2)
- net N$96: no longer names the net of IC14.8 (O), IC17.6 (A3)
- net N$97: no longer names the net of IC14.11 (O), IC17.8 (A4)
- net N$98: no longer names the net of IC15.11 (O), IC17.11 (A1)
- net N$99: no longer names the net of IC15.3 (O), IC17.13 (A2)
Other:
- note removed: "INV-IN[0..7]"
- moved on the sheet: IC16A, IC16B, IC17A, IC17B, IC20A, IC20B, IC23A, IC23B
