File: hardware/cards/bus-tester/kicad/v3.1/bus-tester-v3.1-sheet5.kicad_sch (KiCad schematic)
At the start: 13 parts, among them IC11 74*373, IC12 74*373, IC13 74*373, IC14 74*373, IC15 74*373, IC16 74*373, IC17 74*373, IC18 74*373, IC19 74*373, IC20 74*373, IC21 74*373

Commit message: fix(kicad): readable converted schematics - overlaps 42,847 -> 3,147, nothing off the frame; CF sheet 0 overlaps
- tools/kicad/sch_overlaps.py: calibrated readability check (text/text, text/body, text/line, off frame/title block)
- eagle_sch_to_kicad.py: fields placed from Eagle's smashed attributes or the symbol's >NAME/>VALUE with Eagle's align,
  size and ratio, readable angles; fields Eagle never shows hidden (FABC96R shows only its pin name); pin numbers hidden
  where every Eagle pin hides them; Eagle-hidden layers dropped (the stray SpiceOrder text); labels on their own wires,
  converter labels only where KiCad needs them; rotate-then-mirror fixed for MR90/MR270 in pin_world/no-connects;
  each sheet on the smallest page that holds it, centred clear of the title block
- finish_board.py: stable footprint-library choice (DRC counts no longer vary run to run)
- all 37 projects regenerated: netlist proofs unchanged (34 MATCH, 2 schematic-only, video Fusion export MISMATCH as
  before); DRC same or better; ERC up (loose wire ends onto graphic buses no longer hidden by labels; explained per README)
- CF card: gate names off the gate bodies, U3 clear of its title, 5.08 mm connector pins; rebuilt: DRC 0/0, proof MATCH
- schematic PDFs regenerated (tools/sch_to_pdf.py, 37/37)

Co-Authored-By: Claude Opus 5.5 <noreply@anthropic.com>
Connections:
- net N$30: no longer names the net of -BUS-EN0.3, IC18.5 (2Q)
- net N$48: no longer names the net of -RESET0.3, IC18.9 (4Q)
Other:
- note removed: "BUF-BUS"
- note removed: "BUS"
- moved on the sheet: IC11, IC12, IC13, IC14, IC15, IC16, IC17, IC18, IC19, IC20, IC21
