File: hardware/cards/memory/kicad/deprecated/v1.0/memory-v1.0-sheet5.kicad_sch (KiCad schematic)
At the start: 4 parts, among them IC10 74*00, IC5 74*245

Commit message: fix(kicad): readable converted schematics - overlaps 42,847 -> 3,147, nothing off the frame; CF sheet 0 overlaps
- tools/kicad/sch_overlaps.py: calibrated readability check (text/text, text/body, text/line, off frame/title block)
- eagle_sch_to_kicad.py: fields placed from Eagle's smashed attributes or the symbol's >NAME/>VALUE with Eagle's align,
  size and ratio, readable angles; fields Eagle never shows hidden (FABC96R shows only its pin name); pin numbers hidden
  where every Eagle pin hides them; Eagle-hidden layers dropped (the stray SpiceOrder text); labels on their own wires,
  converter labels only where KiCad needs them; rotate-then-mirror fixed for MR90/MR270 in pin_world/no-connects;
  each sheet on the smallest page that holds it, centred clear of the title block
- finish_board.py: stable footprint-library choice (DRC counts no longer vary run to run)
- all 37 projects regenerated: netlist proofs unchanged (34 MATCH, 2 schematic-only, video Fusion export MISMATCH as
  before); DRC same or better; ERC up (loose wire ends onto graphic buses no longer hidden by labels; explained per README)
- CF card: gate names off the gate bodies, U3 clear of its title, 5.08 mm connector pins; rebuilt: DRC 0/0, proof MATCH
- schematic PDFs regenerated (tools/sch_to_pdf.py, 37/37)

Co-Authored-By: Claude Opus 5.5 <noreply@anthropic.com>
Parts:
- RN3: Eagle name (none) -> RN3_
- RN3: Eagle name (none) -> RN3-8
- RN3: Eagle name (none) -> RN3-2
- RN3: Eagle name (none) -> RN3-4
- RN3: Eagle name (none) -> RN3-3
- RN3: Eagle name (none) -> RN3-7
- RN3: Eagle name (none) -> RN3-1
- RN3: Eagle name (none) -> RN3-6
- RN3: Eagle name (none) -> RN3-5
- RN4: Eagle name (none) -> RN4-1
- RN4: Eagle name (none) -> RN4-8
- RN4: Eagle name (none) -> RN4-2
- RN4: Eagle name (none) -> RN4-4
- RN4: Eagle name (none) -> RN4-6
- RN4: Eagle name (none) -> RN4-3
- RN4: Eagle name (none) -> RN4-5
- RN4: Eagle name (none) -> RN4-7
- RN4: Eagle name (none) -> RN4_
Connections:
- net N$12: no longer names the net of IC10.1 (I0), IC10.2 (I1), IC10.6 (O)
- net N$13: no longer names the net of IC10.3 (O), IC5.19 (G)
Other:
- note removed: "BDATA0,BDATA1,BDATA2,BDATA3,BDATA4,BDATA5,BDATA6,BDATA7"
- note removed: "DATA[0..7]"
- moved on the sheet: IC5
