File: hardware/cards/memory/kicad/deprecated/v1.1/memory-v1.1-sheet3.kicad_sch (KiCad schematic)
At the start: 4 parts, among them IC1 62256P, IC2 62256P, IC3 2732, IC6 74*04

Commit message: fix(kicad): readable converted schematics - overlaps 42,847 -> 3,147, nothing off the frame; CF sheet 0 overlaps
- tools/kicad/sch_overlaps.py: calibrated readability check (text/text, text/body, text/line, off frame/title block)
- eagle_sch_to_kicad.py: fields placed from Eagle's smashed attributes or the symbol's >NAME/>VALUE with Eagle's align,
  size and ratio, readable angles; fields Eagle never shows hidden (FABC96R shows only its pin name); pin numbers hidden
  where every Eagle pin hides them; Eagle-hidden layers dropped (the stray SpiceOrder text); labels on their own wires,
  converter labels only where KiCad needs them; rotate-then-mirror fixed for MR90/MR270 in pin_world/no-connects;
  each sheet on the smallest page that holds it, centred clear of the title block
- finish_board.py: stable footprint-library choice (DRC counts no longer vary run to run)
- all 37 projects regenerated: netlist proofs unchanged (34 MATCH, 2 schematic-only, video Fusion export MISMATCH as
  before); DRC same or better; ERC up (loose wire ends onto graphic buses no longer hidden by labels; explained per README)
- CF card: gate names off the gate bodies, U3 clear of its title, 5.08 mm connector pins; rebuilt: DRC 0/0, proof MATCH
- schematic PDFs regenerated (tools/sch_to_pdf.py, 37/37)

Co-Authored-By: Claude Opus 5.5 <noreply@anthropic.com>
Connections:
- net MEM-RD: no longer names the net of IC6.1 (I), IC6.6 (O)
- net N$2: no longer names the net of IC6.3 (I), IC6.8 (O)
- net N$3: no longer names the net of IC1.22 (~{OE}), IC2.22 (~{OE}), IC3.20 (~{OE}/VPP), IC6.2 (O)
- net N$4: no longer names the net of IC1.27 (~{WE}), IC2.27 (~{WE}), IC6.4 (O)
Other:
- note removed: "BADDR[0..15]"
- note removed: "BDATA[0..7]"
- moved on the sheet: IC1, IC2, IC3
