File: hardware/cards/register/kicad/deprecated/v1.0-no-address/register-v1.0-no-address-sheet8.kicad_sch (KiCad schematic)
At the start: 5 parts, among them IC31 74*32, IC35 74*245, IC36 74*245, IC37 74*245, IC38 74*266

Commit message: fix(kicad): readable converted schematics - overlaps 42,847 -> 3,147, nothing off the frame; CF sheet 0 overlaps
- tools/kicad/sch_overlaps.py: calibrated readability check (text/text, text/body, text/line, off frame/title block)
- eagle_sch_to_kicad.py: fields placed from Eagle's smashed attributes or the symbol's >NAME/>VALUE with Eagle's align,
  size and ratio, readable angles; fields Eagle never shows hidden (FABC96R shows only its pin name); pin numbers hidden
  where every Eagle pin hides them; Eagle-hidden layers dropped (the stray SpiceOrder text); labels on their own wires,
  converter labels only where KiCad needs them; rotate-then-mirror fixed for MR90/MR270 in pin_world/no-connects;
  each sheet on the smallest page that holds it, centred clear of the title block
- finish_board.py: stable footprint-library choice (DRC counts no longer vary run to run)
- all 37 projects regenerated: netlist proofs unchanged (34 MATCH, 2 schematic-only, video Fusion export MISMATCH as
  before); DRC same or better; ERC up (loose wire ends onto graphic buses no longer hidden by labels; explained per README)
- CF card: gate names off the gate bodies, U3 clear of its title, 5.08 mm connector pins; rebuilt: DRC 0/0, proof MATCH
- schematic PDFs regenerated (tools/sch_to_pdf.py, 37/37)

Co-Authored-By: Claude Opus 5.5 <noreply@anthropic.com>
Connections:
- net N$1: no longer names the net of IC31.8 (O), IC35.19 (G), IC36.19 (G)
- net N$37: no longer names the net of IC31.11 (O), IC37.19 (G)
- net N$41: no longer names the net of IC31.9 (I0), IC38.4 (O)
- net N$42: no longer names the net of IC31.10 (I1), IC31.12 (I0), IC38.11 (O)
Other:
- note removed: "ADATA[0..7]"
- note removed: "ADATA[8..15]"
- note removed: "DATA[0..7]"
- note removed: "DATA[8..15]"
- moved on the sheet: IC35, IC36, IC37
