File: hardware/cards/register/kicad/deprecated/v1.0-no-address/register-v1.0-no-address-sheet9.kicad_sch (KiCad schematic)
At the start: 3 parts, among them X1 FABC96R

Commit message: fix(kicad): readable converted schematics - overlaps 42,847 -> 3,147, nothing off the frame; CF sheet 0 overlaps
- tools/kicad/sch_overlaps.py: calibrated readability check (text/text, text/body, text/line, off frame/title block)
- eagle_sch_to_kicad.py: fields placed from Eagle's smashed attributes or the symbol's >NAME/>VALUE with Eagle's align,
  size and ratio, readable angles; fields Eagle never shows hidden (FABC96R shows only its pin name); pin numbers hidden
  where every Eagle pin hides them; Eagle-hidden layers dropped (the stray SpiceOrder text); labels on their own wires,
  converter labels only where KiCad needs them; rotate-then-mirror fixed for MR90/MR270 in pin_world/no-connects;
  each sheet on the smallest page that holds it, centred clear of the title block
- finish_board.py: stable footprint-library choice (DRC counts no longer vary run to run)
- all 37 projects regenerated: netlist proofs unchanged (34 MATCH, 2 schematic-only, video Fusion export MISMATCH as
  before); DRC same or better; ERC up (loose wire ends onto graphic buses no longer hidden by labels; explained per README)
- CF card: gate names off the gate bodies, U3 clear of its title, 5.08 mm connector pins; rebuilt: DRC 0/0, proof MATCH
- schematic PDFs regenerated (tools/sch_to_pdf.py, 37/37)

Co-Authored-By: Claude Opus 5.5 <noreply@anthropic.com>
Parts:
- X1: Eagle name (none) -> X1-B4
- X1: Eagle name (none) -> X1-C27
- X1: Eagle name (none) -> X1-B30
- X1: Eagle name (none) -> X1-B26
- X1: Eagle name (none) -> X1-B31
- X1: Eagle name (none) -> X1-A9
- X1: Eagle name (none) -> X1-A6
- X1: Eagle name (none) -> X1-B20
- X1: Eagle name (none) -> X1-C13
- X1: Eagle name (none) -> X1-B21
- X1: Eagle name (none) -> X1-A18
- X1: Eagle name (none) -> X1-A10
- X1: Eagle name (none) -> X1-C6
- X1: Eagle name (none) -> X1-B3
- X1: Eagle name (none) -> X1-C9
- X1: Eagle name (none) -> X1-B1
- X1: Eagle name (none) -> X1-B14
- X1: Eagle name (none) -> X1-C8
- X1: Eagle name (none) -> X1-C15
- X1: Eagle name (none) -> X1-A26
- X1: Eagle name (none) -> X1-A7
- X1: Eagle name (none) -> X1-C20
- X1: Eagle name (none) -> X1-A8
- X1: Eagle name (none) -> X1-B22
- X1: Eagle name (none) -> X1-B23
- X1: Eagle name (none) -> X1-A2
- X1: Eagle name (none) -> X1-A22
- X1: Eagle name (none) -> X1-A5
- X1: Eagle name (none) -> X1-B11
- X1: Eagle name (none) -> X1-A15
- X1: Eagle name (none) -> X1-B6
- X1: Eagle name (none) -> X1-A12
- X1: Eagle name (none) -> X1-A17
- X1: Eagle name (none) -> X1-A32
- X1: Eagle name (none) -> X1-C3
- X1: Eagle name (none) -> X1-C29
- X1: Eagle name (none) -> X1-C5
- X1: Eagle name (none) -> X1-A1
- X1: Eagle name (none) -> X1-A4
- X1: Eagle name (none) -> X1-C24
- X1: Eagle name (none) -> X1-C4
- X1: Eagle name (none) -> X1-C21
- X1: Eagle name (none) -> X1-A11
- X1: Eagle name (none) -> X1-A29
- X1: Eagle name (none) -> X1-C10
- X1: Eagle name (none) -> X1-B32
- X1: Eagle name (none) -> X1-C31
- X1: Eagle name (none) -> X1-A25
- X1: Eagle name (none) -> X1-B8
- X1: Eagle name (none) -> X1-B27
- X1: Eagle name (none) -> X1-B28
- X1: Eagle name (none) -> X1-C28
- X1: Eagle name (none) -> X1-C19
- X1: Eagle name (none) -> X1-A3
- X1: Eagle name (none) -> X1-B25
- X1: Eagle name (none) -> X1-C22
- X1: Eagle name (none) -> X1-B17
- X1: Eagle name (none) -> X1-A27
- X1: Eagle name (none) -> X1-C7
- X1: Eagle name (none) -> X1-B5
- X1: Eagle name (none) -> X1-B16
- X1: Eagle name (none) -> X1-B29
- X1: Eagle name (none) -> X1-C17
- X1: Eagle name (none) -> X1-B12
- X1: Eagle name (none) -> X1-C25
- X1: Eagle name (none) -> X1-A23
- X1: Eagle name (none) -> X1-C12
- X1: Eagle name (none) -> X1-C23
- X1: Eagle name (none) -> X1-A21
- X1: Eagle name (none) -> X1-B24
- X1: Eagle name (none) -> X1-A31
- X1: Eagle name (none) -> X1-C32
- X1: Eagle name (none) -> X1-A19
- X1: Eagle name (none) -> X1-B13
- X1: Eagle name (none) -> X1-B10
- X1: Eagle name (none) -> X1-C18
- X1: Eagle name (none) -> X1-B7
- X1: Eagle name (none) -> X1-C16
- X1: Eagle name (none) -> X1-C14
- X1: Eagle name (none) -> X1-C26
- X1: Eagle name (none) -> X1-C30
- X1: Eagle name (none) -> X1-A14
- X1: Eagle name (none) -> X1-A20
- X1: Eagle name (none) -> X1-B9
- X1: Eagle name (none) -> X1-B15
- X1: Eagle name (none) -> X1-A30
- X1: Eagle name (none) -> X1-B2
- X1: Eagle name (none) -> X1-B19
- X1: Eagle name (none) -> X1-C2
- X1: Eagle name (none) -> X1-C11
- X1: Eagle name (none) -> X1-A13
- X1: Eagle name (none) -> X1-A24
- X1: Eagle name (none) -> X1-B18
- X1: Eagle name (none) -> X1-A16
- X1: Eagle name (none) -> X1-C1
- X1: Eagle name (none) -> X1-A28
Connections:
- net N$44: no longer names the net of PWR0.A, R1.1
Other:
- note removed: "-AC-LD,-AC-LD-INV,-AC-RD,ADDR[0..15],-ADDR-REG-LD[0..1],-ADDR-REG-RD[0..1],ALU[0..3],-ALU-FUNC,BR-COND,-BUS-EN,DATA[0..15],-HL-SWAP,IN,-INT,-INTA,IO-ADDR[0..3],-IO-ADDR-LD,-IO-RD,-IO-WR,-MEM-RD,-MEM-WR,OUT,-REG-DN,-REG-FUNC-LD,-REG-FUNC-RD,-REG-LD-HI,REG-LD-ID[0..3],-REG-LD-LO,-REG-RD-HI,REG-RD-ID[0..3],-REG-RD-LO,-REG-UP,-RESET,-RUN,-SR-LD,-TMP-REG-LD[0..1],-TMP-REG-RD[0..1],UNUSED0"
