File: hardware/cards/sequencer-logic/kicad/v2.1/orig-size/sequencer-logic-prod-v2.1-copy/sequencer-logic-v2.1-orig-size-sequencer-logic-prod-v2.1-copy-sheet1.kicad_sch (KiCad schematic)
At the start: 19 parts, among them IC1 74*244, IC10 74*32, IC11 74*04, IC12 74*08, IC2 74*244, IC22 74*74, IC23 74*02, IC29 74*08, IC3 74*175, IC30 74*04, IC35 74*32, IC36 74*04, IC4 74*175, IC5 74*192, IC6 74*192, IC7 74*08, IC8 74*244, IC9 74*244

Commit message: fix(kicad): readable converted schematics - overlaps 42,847 -> 3,147, nothing off the frame; CF sheet 0 overlaps
- tools/kicad/sch_overlaps.py: calibrated readability check (text/text, text/body, text/line, off frame/title block)
- eagle_sch_to_kicad.py: fields placed from Eagle's smashed attributes or the symbol's >NAME/>VALUE with Eagle's align,
  size and ratio, readable angles; fields Eagle never shows hidden (FABC96R shows only its pin name); pin numbers hidden
  where every Eagle pin hides them; Eagle-hidden layers dropped (the stray SpiceOrder text); labels on their own wires,
  converter labels only where KiCad needs them; rotate-then-mirror fixed for MR90/MR270 in pin_world/no-connects;
  each sheet on the smallest page that holds it, centred clear of the title block
- finish_board.py: stable footprint-library choice (DRC counts no longer vary run to run)
- all 37 projects regenerated: netlist proofs unchanged (34 MATCH, 2 schematic-only, video Fusion export MISMATCH as
  before); DRC same or better; ERC up (loose wire ends onto graphic buses no longer hidden by labels; explained per README)
- CF card: gate names off the gate bodies, U3 clear of its title, 5.08 mm connector pins; rebuilt: DRC 0/0, proof MATCH
- schematic PDFs regenerated (tools/sch_to_pdf.py, 37/37)

Co-Authored-By: Claude Opus 5.5 <noreply@anthropic.com>
Connections:
- net COUNT-RESET: no longer names the net of IC10.3 (O), IC5.14 (CLR), IC6.14 (CLR)
- net N$1: no longer names the net of IC5.5 (UP), IC6.12 (CO)
- net N$10: no longer names the net of IC1.6 (A3), IC4.10 (Q3)
- net N$11: no longer names the net of IC2.8 (A4), IC6.7 (QD)
- net N$12: no longer names the net of IC2.11 (A1), IC5.3 (QA)
- net N$13: no longer names the net of IC2.13 (A2), IC5.2 (QB)
- net N$14: no longer names the net of IC2.15 (A3), IC5.6 (QC)
- net N$15: no longer names the net of IC2.17 (A4), IC5.7 (QD)
- net N$16: no longer names the net of IC36.6 (O), IC7.1 (I0)
- net N$17: no longer names the net of IC4.12 (D3), IC8.14 (Y3), IC9.14 (Y3)
- net N$18: no longer names the net of IC4.13 (D4), IC8.12 (Y4), IC9.12 (Y4)
- net N$19: no longer names the net of IC3.4 (D1), IC8.9 (Y1), IC9.9 (Y1)
- net N$2: no longer names the net of IC1.2 (A1), IC4.2 (Q1)
- net N$20: no longer names the net of IC3.5 (D2), IC8.7 (Y2), IC9.7 (Y2)
- net N$21: no longer names the net of IC3.12 (D3), IC8.5 (Y3), IC9.5 (Y3)
- net N$22: no longer names the net of IC3.13 (D4), IC8.3 (Y4), IC9.3 (Y4)
- net N$23: no longer names the net of IC1.8 (A4), IC4.15 (Q4)
- net N$26: no longer names the net of IC10.11 (O), IC36.5 (I)
- net N$3: no longer names the net of IC1.4 (A2), IC4.7 (Q2)
- net N$31: no longer names the net of IC7.3 (O), IC7.4 (I0)
- net N$32: no longer names the net of IC23.10 (O), IC35.12 (I0)
- net N$33: no longer names the net of IC22.11 (CLK), IC35.6 (O)
- net N$34: no longer names the net of IC1.11 (A1), IC3.2 (Q1)
- net N$35: no longer names the net of IC1.13 (A2), IC3.7 (Q2)
- net N$36: no longer names the net of IC1.15 (A3), IC3.10 (Q3)
- net N$37: no longer names the net of IC1.17 (A4), IC3.15 (Q4)
- net N$38: no longer names the net of IC10.5 (I1), IC7.11 (O)
- net N$39: no longer names the net of IC10.4 (I0), IC7.8 (O)
- net N$4: no longer names the net of IC29.5 (I1), IC6.5 (UP), IC7.6 (O)
- net N$40: no longer names the net of IC7.9 (I0), QG1.8 (OUT)
- net N$42: no longer names the net of IC11.11 (I), IC30.8 (O)
- net N$44: no longer names the net of IC30.2 (O), IC30.9 (I)
- net N$46: no longer names the net of IC11.10 (O), IC23.9 (I1)
- net N$5: no longer names the net of IC4.4 (D1), IC8.18 (Y1), IC9.18 (Y1)
- net N$54: no longer names the net of IC12.11 (O), IC35.4 (I0)
- net N$55: no longer names the net of IC10.2 (I1), IC29.6 (O)
- net N$6: no longer names the net of IC4.5 (D2), IC8.16 (Y2), IC9.16 (Y2)
- net N$7: no longer names the net of IC2.2 (A1), IC6.3 (QA)
- net N$8: no longer names the net of IC2.4 (A2), IC6.2 (QB)
- net N$9: no longer names the net of IC2.6 (A3), IC6.6 (QC)
Other:
- moved on the sheet: IC1A, IC1B, IC22B, IC2A, IC2B, IC3, IC4, IC5, IC6, IC8A, IC8B, IC9A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
