File: hardware/cards/memory/kicad/v2.0/memory-v2.0-option-b.kicad_pcb (KiCad board)
At the start: 4 copper layers, 177.8 x 114 mm, 73 parts, among them IC10 74ALS00N, IC11 74LS157N, IC12 74LS74N, IC14 74LS04N, IC18 74ALS30N, IC26 74LS374N, IC27 74LS374N, IC28 74LS374N, IC29 74LS374N, IC3 74LS32N, IC30 74LS138, IC31 74LS32, IC32 74LS175, IC33 74LS08, IC34 74LS245, IC4 74ALS30N, IC5 74LS245N, IC6 74LS04N, IC7 74LS138N, IC8 74LS244N, IC9 74LS244N, J2 IDE 40, J3 POWER, X1 FABC96R

Commit message: feat(memory): rebuild memory card v2.0 on the built card - CF section does not fit, placement blocked
hardware/cards/memory/kicad/v2.0 is now generated from ../v1.3-fusion-export-2026-09-24 (the built
card) instead of the earlier save: v2.0 = built card + the CF section (CF card v1.0 circuit on P8/P9,
IC30-IC34, J2/J3/JP2, RN9, R10-R14, LED1, C25-C30), IC15 included with its real wiring. Netlist proof
MATCH pin for pin (74 parts, 186 nets; every option board = the schematic); ERC 99 = the built
card's 104 + SRST - the six labels made global.

The built card's copper is locked: gen_mem_v2.py no longer trims or drops copper, it refuses moves
that would break a track, and "locked" proves all 1377 track segments/vias present unchanged on
every board. FAB_MOVES and the reserved IC15 spot are gone (the parts are simply the built card's).
The built card's Eagle rules that are stricter than the project's go into memory-v2.0.kicad_dru
(18 mil track-track, 10 mil track-pad). build.sh now gates on the summary files (a pipeline hid
failed gates before).

Result: the built card routes DATA8-15 to the TMP registers as a bundle across the lower right of
the board, through the slots the three options used. Every option has CF pads on built tracks
(A 11 shorts / 4 clearance / 63 mask bridges, B 12/1/50, C 12/3/63). space_check.py shows no legal
placement exists: at most 4 of the 5 CF DIPs fit even with no IDE header and none of the other 16
CF parts (2 with J2 where option C puts it). Not routed, not ordered; README lists the ways forward
(re-route that bundle, keep the separate CF card, SMD CF logic, or a new layout). Docs and BACKLOG
say v2.0 is blocked.

Co-Authored-By: Claude Opus 5.5 <noreply@anthropic.com>
Parts:
- added IC15: 74ALS11N, memory-v1.3-fusion-export-2026-09-24-eagle:DIL14, F.Cu at (168.9, 70.7)
- C1, C10, C11, C12, C13, C14, C15, C16, C17, C18, C19, C2, C20, C21, C22, C23, C24, C3, C4, C5, C6, C7, C8, C9: footprint memory-v1.3-eagle:C025-025X050 -> memory-v1.3-fusion-export-2026-09-24-eagle:C025-025X050
- IC1, IC13, IC2: footprint memory-v1.3-eagle:DIL28-6 -> memory-v1.3-fusion-export-2026-09-24-eagle:DIL28-6
- IC10, IC12, IC14, IC18, IC3, IC4, IC6: footprint memory-v1.3-eagle:DIL14 -> memory-v1.3-fusion-export-2026-09-24-eagle:DIL14
- IC11, IC7: footprint memory-v1.3-eagle:DIL16 -> memory-v1.3-fusion-export-2026-09-24-eagle:DIL16
- IC26, IC27, IC28, IC29, IC5, IC8, IC9: footprint memory-v1.3-eagle:DIL20 -> memory-v1.3-fusion-export-2026-09-24-eagle:DIL20
- JP1: footprint memory-v1.3-eagle:1X03 -> memory-v1.3-fusion-export-2026-09-24-eagle:1X03
- PWR0: footprint memory-v1.3-eagle:LED5MM -> memory-v1.3-fusion-export-2026-09-24-eagle:LED5MM
- R2: footprint memory-v1.3-eagle:0207_10 -> memory-v1.3-fusion-export-2026-09-24-eagle:0207_10
- RN5, RN6: footprint memory-v1.3-eagle:RN-9 -> memory-v1.3-fusion-export-2026-09-24-eagle:RN-9
- RN7, RN8: footprint memory-v1.3-eagle:SIL9 -> memory-v1.3-fusion-export-2026-09-24-eagle:SIL9
- U$1: footprint memory-v1.3-eagle:PIN_3X8 -> memory-v1.3-fusion-export-2026-09-24-eagle:PIN_3X8
- X1: footprint memory-v1.3-eagle:FABC96R -> memory-v1.3-fusion-export-2026-09-24-eagle:FABC96R
Connections:
- net /Sheet 3/-LO-RAM renamed -LO-RAM
- net Net-(IC18-I0) renamed /Sheet 2/ROM7
- net Net-(IC18-I1) renamed /Sheet 2/ROM6
- net Net-(IC18-I2) renamed /Sheet 2/ROM5
- net Net-(IC18-I3) renamed /Sheet 2/ROM4
- net Net-(IC18-I4) renamed /Sheet 2/ROM3
- net Net-(IC18-I5) renamed /Sheet 2/ROM2
- net Net-(IC18-I6) renamed /Sheet 2/ROM1
- net Net-(IC18-I7) renamed /Sheet 2/ROM0
- net Net-(IC4-I0) renamed /Sheet 2/RAM0
- net Net-(IC4-I1) renamed /Sheet 2/RAM1
- net Net-(IC4-I2) renamed /Sheet 2/RAM2
- net Net-(IC4-I3) renamed /Sheet 2/RAM3
- net Net-(IC4-I4) renamed /Sheet 2/RAM4
- net Net-(IC4-I5) renamed /Sheet 2/RAM5
- net Net-(IC4-I6) renamed /Sheet 2/RAM6
- net Net-(IC4-I7) renamed /Sheet 2/RAM7
- net Net-(IC7-Y0) renamed /Sheet 2/SEL0
- net Net-(IC7-Y1) renamed /Sheet 2/SEL1
- net Net-(IC7-Y2) renamed /Sheet 2/SEL2
- net Net-(IC7-Y3) renamed /Sheet 2/SEL3
- net Net-(IC7-Y4) renamed /Sheet 2/SEL4
- net Net-(IC7-Y5) renamed /Sheet 2/SEL5
- net Net-(IC7-Y6) renamed /Sheet 2/SEL6
- net Net-(IC7-Y7) renamed /Sheet 2/SEL7
- IC5 pad 19: -VMA -> Net-(IC15A-O)
Routing:
- net DATA11: track 2.54 -> 365.5 mm, vias 0 -> 2
- net DATA9: track 0.00 -> 309.2 mm, vias 0 -> 2
- net DATA10: track 0.00 -> 295.8 mm, vias 0 -> 3
- net DATA8: track 0.00 -> 256.7 mm, vias 0 -> 1
- net DATA12: track 0.00 -> 248.0 mm, vias 0 -> 1
- net DATA13: track 0.00 -> 244.3 mm, vias 0 -> 1
- net DATA15: track 0.00 -> 234.9 mm, vias 0 -> 1
- net DATA14: track 0.00 -> 231.2 mm, vias 0 -> 2
- net Net-(IC14A-O): track 0.00 -> 211.2 mm, vias 0 -> 2
- net DATA4: track 72.3 -> 281.7 mm, vias 1 -> 3
- net DATA7: track 89.0 -> 296.2 mm, vias 1 -> 3
- net DATA1: track 54.7 -> 261.4 mm, vias 0 -> 5
- net DATA3: track 73.8 -> 278.6 mm, vias 1 -> 2
- net DATA5: track 71.9 -> 269.2 mm, vias 1 -> 4
- net DATA6: track 81.8 -> 264.6 mm, vias 1 -> 4
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Other:
- board text added: "0X8000"
- board text added: "0XF000"
- board text added: "RAM"
- board text added: "ROM"
- board text removed: "fabricated card only,"
- board text removed: "not in the v1.3 schematic"
- board text removed: "reserved: IC15 74ALS11"
