File: hardware/cards/memory/kicad/v2.0/memory-v2.0-relayout-c.kicad_pcb (KiCad board)
At the start: 4 copper layers, 177.8 x 114 mm, 74 parts, among them IC10 74ALS00N, IC11 74LS157N, IC12 74LS74N, IC14 74LS04N, IC15 74ALS11N, IC18 74ALS30N, IC26 74LS374N, IC27 74LS374N, IC28 74LS374N, IC29 74LS374N, IC3 74LS32N, IC30 74LS138, IC31 74LS32, IC32 74LS175, IC33 74LS08, IC34 74LS245, IC4 74ALS30N, IC5 74LS245N, IC6 74LS04N, IC7 74LS138N, IC8 74LS244N, IC9 74LS244N, J2 IDE 40, J3 POWER, X1 FABC96R

Commit message: refactor(memory): built card is eagle/v1.3; the earlier save is eagle/deprecated/v1.3-do-not-use
Ken 2026-09-24: the memory card folders are renamed so the plain v1.3 name is the card in the machine.

- eagle/v1.3/ (earlier save, notes 2025-03-06, board 2021-03-17, NOT the built card) -> eagle/deprecated/v1.3-do-not-use/
  (git mv, contents untouched); its KiCad conversion regenerated as kicad/deprecated/v1.3-do-not-use/ (project
  memory-v1.3-do-not-use, proof MATCH 115/115, still "never fabricated").
- eagle/v1.3-fusion-export-2026-09-24/ (the BUILT card: Ken's Fusion 360 export of 2026-09-24, verified against JLCPCB
  order 2000765A) -> eagle/v1.3/; its conversion regenerated as kicad/v1.3/ (memory-v1.3.*, proof MATCH 116/116).
  verify_fab_vs_brd.py: PASS on eagle/v1.3 (all 695 holes, 1,263 tracks, parts, PnP; gerber set byte-identical to
  the one kept in the deprecated folder), FAIL on the deprecated board as before.
- Migration plan: tools/migrate_dryrun.py sends GV "Memory v1.3" to eagle/deprecated/v1.3-do-not-use/; migration/
  reports re-run (the 30 plan rows differ only by that destination). audit_tree.py: the Fusion-export rule now
  matches eagle/v1.3/ and is checked before the 2026-09-20 run log (which lists the earlier save at that path).
  Audit: 0 unexplained, 0 hash mismatches, 0 plan rows missing.
- fabricated.py -> FABRICATED.md + marker, gen_bom.py (+ docs/bom rows, --check up to date), PROVENANCE.md
  regenerated, KICAD.md rows (stale fusion-export row removed), BOARDS.md/SCHEMATICS.md rows, the memory section of
  DESIGN-REVIEW.md (now the built card: 53 parts, 169 nets, 21 ICs; the rest of that file is left at its 09-21 run).
- memory v2.0 reads ../v1.3: BASE_NAME/BASE/space_check path/docstrings/MASTER/README. The copied library is renamed
  memory-v1.3-eagle (the regenerated base's nickname; gen_mem_v2.py sch copies it with the lib tables). The converter
  derives schematic UUIDs from the project name, so in the boards a NOROUTE build does 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
Parts:
- C1, C10, C11, C12, C13, C14, C15, C16, C17, C18, C19, C2, C20, C21, C22, C23, C24, C3, C4, C5, C6, C7, C8, C9: footprint memory-v1.3-fusion-export-2026-09-24-eagle:C025-025X050 -> memory-v1.3-eagle:C025-025X050
- IC1, IC13, IC2: footprint memory-v1.3-fusion-export-2026-09-24-eagle:DIL28-6 -> memory-v1.3-eagle:DIL28-6
- IC10, IC12, IC14, IC15, IC18, IC3, IC4, IC6: footprint memory-v1.3-fusion-export-2026-09-24-eagle:DIL14 -> memory-v1.3-eagle:DIL14
- IC11, IC7: footprint memory-v1.3-fusion-export-2026-09-24-eagle:DIL16 -> memory-v1.3-eagle:DIL16
- IC26, IC27, IC28, IC29, IC5, IC8, IC9: footprint memory-v1.3-fusion-export-2026-09-24-eagle:DIL20 -> memory-v1.3-eagle:DIL20
- JP1: footprint memory-v1.3-fusion-export-2026-09-24-eagle:1X03 -> memory-v1.3-eagle:1X03
- PWR0: footprint memory-v1.3-fusion-export-2026-09-24-eagle:LED5MM -> memory-v1.3-eagle:LED5MM
- R2: footprint memory-v1.3-fusion-export-2026-09-24-eagle:0207_10 -> memory-v1.3-eagle:0207_10
- RN5, RN6: footprint memory-v1.3-fusion-export-2026-09-24-eagle:RN-9 -> memory-v1.3-eagle:RN-9
- RN7, RN8: footprint memory-v1.3-fusion-export-2026-09-24-eagle:SIL9 -> memory-v1.3-eagle:SIL9
- U$1: footprint memory-v1.3-fusion-export-2026-09-24-eagle:PIN_3X8 -> memory-v1.3-eagle:PIN_3X8
- X1: footprint memory-v1.3-fusion-export-2026-09-24-eagle:FABC96R -> memory-v1.3-eagle:FABC96R
