File: hardware/cards/memory/kicad/v2.0/memory-v2.0-sheet1.kicad_sch (KiCad schematic)
At the start: 30 parts, among them IC12 74*74, IC15 74*11, IC3 74*32, X1 FABC96R

Commit message: feat(memory): remove C20-C23 from memory card v2.0 - the four 100 nF with no IC beside them
Ken, 2026-09-24: "get rid of unused capacitors on the memory card". C20-C23 were the
built card's spare plane-to-plane caps (pin 1 GND, pin 2 VCC, nothing else); every IC
keeps its own 100 nF (C1-C19, C24, C25-C29) and C30 (10 uF at J3) stays.

- mem_v2_netlist.REMOVED is the single source; expected() checks each was a plain
  VCC-GND cap on v1.3 and takes it out: v2.0 = v1.3 - C20-C23 + CF (70 parts, 687 pins)
- gen_mem_v2.py sch: remove_parts() drops the symbols from sheet 1's cap row, merges
  the GND/VCC rail wires C19-C24 and removes the junctions; ERC unchanged (99, PASS)
- check_netlist.py: final board must equal the schematic; --records boards (options,
  trial routes, keep-copper, made before the removal and left as they were) must equal
  the schematic + exactly C20-C23 as on v1.3; anything else fails
- finish_v2.py make: drop_removed() after the silk tidy, then refill; the committed board
  re-made this way: only the four footprints gone + planes refilled, no track or via
  touched them, routing unchanged (43 vias, 11,779 mm), DRC 0 copper, 174 power pads
  on solid planes; FROM=trial reproduces it
- generators keep the four on regenerated records; build.sh parity accepts them there only
- fab outputs, schematic PDF, BOM (70 parts), reports regenerated; README, KICAD.md,
  docs/cards/memory.md, BACKLOG updated

Co-Authored-By: Claude Opus 5.5 <noreply@anthropic.com>
Parts:
- removed C20, C21, C22, C23: C-US, memory-v1.3-eagle:C025-025X050, symbol memory-v1.3-eagle:adafruit_C-US_025-025X050
Other:
- note added: "Memory card v2.0: IO-ADDR0-3 (C7-C10), -IO-RD (B25), -IO-WR (B26) and -RESET (C30) also feed the CompactFlash section on sheet 7 (I/O ports P8 = register latch, P9 = data; its own 74LS138 IC30, enabled by IO-ADDR3). DATA0-7 reach its data buffer IC34 and latch IC32. v1.3 used none of the I/O signals: the six labels above were X1-only local labels and are global labels now. C20-C23 (v1.3: four 100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"
- note removed: "Memory card v2.0: IO-ADDR0-3 (C7-C10), -IO-RD (B25), -IO-WR (B26) and -RESET (C30) also feed the CompactFlash section on sheet 7 (I/O ports P8 = register latch, P9 = data; its own 74LS138 IC30, enabled by IO-ADDR3). DATA0-7 reach its data buffer IC34 and latch IC32. v1.3 used none of the I/O signals: the six labels above were X1-only local labels and are global labels now."
Changed lines of the file:
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@@
 	(generator_version "1.0")
 	(paper "A3")
-	(title_block (title "memory-v2.0 sheet 1") (date "2026-09-24") (rev "v2.0") (comment 1 "v1.3 sheet 1 + IO-ADDR0-3, -IO-RD, -IO-WR made global (CF section, sheet 7) + note"))
+	(title_block (title "memory-v2.0 sheet 1") (date "2026-09-24") (rev "v2.0") (comment 1 "v1.3 sheet 1: 6 bus labels global (CF, sheet 7), C20-C23 removed, + note"))
 	(symbol (lib_id "memory-v1.3-eagle:con-vg_FABC96R") (at 101.6 172.72 90) (unit 3)
 		(exclude_from_sim no) (in_bom yes) (on_board yes) (dnp no)
@@
 		(pin "2")
 		(instances (project "memory-v2.0" (path "/42231b4d-4c5f-cebb-da74-8d622a2f1dd4/36727bec-ef3f-c35c-0354-2dfce4bdbefc" (reference "C19") (unit 1))))
-	)
-	(symbol (lib_id "memory-v1.3-eagle:adafruit_C-US_025-025X050") (at 241.3 97.79 0) (unit 1)
-		(exclude_from_sim no) (in_bom yes) (on_board yes) (dnp no)
-		(property "Reference" "C20" (at 242.316 97.155 0) (effects (font (size 1.778 1.778) (thickness 0.1422)) (justify left bottom)))
-		(property "Value" "C-US" (at 242.316 101.981 0) (effects (font (size 1.778 1.778) (thickness 0.1422)) (justify left bottom)))
-		(property "Footprint" "memory-v1.3-eagle:C025-025X050" (at 241.3 97.79 0) (effects (font (size 1.27 1.27)) (hide yes)))
-		(property "Datasheet" "" (at 241.3 97.79 0) (effects (font (size 1.27 1.27)) (hide yes)))
-		(pin "1")
-		(pin "2")
-		(instances (project "memory-v2.0" (path "/42231b4d-4c5f-cebb-da74-8d622a2f1dd4/36727bec-ef3f-c35c-0354-2dfce4bdbefc" (reference "C20") (unit 1))))
-	)
-	(symbol (lib_id "memory-v1.3-eagle:adafruit_C-US_025-025X050") (at 248.92 97.79 0) (unit 1)
-		(exclude_from_sim no) (in_bom yes) (on_board yes) (dnp no)
-		(property "Reference" "C21" (at 249.936 97.155 0) (effects (font (size 1.778 1.778) (thickness 0.1422)) (justify left bottom)))
-		(property "Value" "C-US" (at 249.936 101.981 0) (effects (font (size 1.778 1.778) (thickness 0.1422)) (justify left bottom)))
-		(property "Footprint" "memory-v1.3-eagle:C025-025X050" (at 248.92 97.79 0) (effects (font (size 1.27 1.27)) (hide yes)))
-		(property "Datasheet" "" (at 248.92 97.79 0) (effects (font (size 1.27 1.27)) (hide yes)))
-		(pin "1")
-		(pin "2")
-		(instances (project "memory-v2.0" (path "/42231b4d-4c5f-cebb-da74-8d622a2f1dd4/36727bec-ef3f-c35c-0354-2dfce4bdbefc" (reference "C21") (unit 1))))
-	)
-	(symbol (lib_id "memory-v1.3-eagle:adafruit_C-US_025-025X050") (at 256.54 97.79 0) (unit 1)
-		(exclude_from_sim no) (in_bom yes) (on_board yes) (dnp no)
-		(property "Reference" "C22" (at 257.556 97.155 0) (effects (font (size 1.778 1.778) (thickness 0.1422)) (justify left bottom)))
-		(property "Value" "C-US" (at 257.556 101.981 0) (effects (font (size 1.778 1.778) (thickness 0.1422)) (justify left bottom)))
-		(property "Footprint" "memory-v1.3-eagle:C025-025X050" (at 256.54 97.79 0) (effects (font (size 1.27 1.27)) (hide yes)))
-		(property "Datasheet" "" (at 256.54 97.79 0) (effects (font (size 1.27 1.27)) (hide yes)))
-		(pin "1")
-		(pin "2")
-		(instances (project "memory-v2.0" (path "/42231b4d-4c5f-cebb-da74-8d622a2f1dd4/36727bec-ef3f-c35c-0354-2dfce4bdbefc" (reference "C22") (unit 1))))
-	)
-	(symbol (lib_id "memory-v1.3-eagle:adafruit_C-US_025-025X050") (at 264.16 97.79 0) (unit 1)
-		(exclude_from_sim no) (in_bom yes) (on_board yes) (dnp no)
-		(property "Reference" "C23" (at 265.176 97.155 0) (effects (font (size 1.778 1.778) (thickness 0.1422)) (justify left bottom)))
-		(property "Value" "C-US" (at 265.176 101.981 0) (effects (font (size 1.778 1.778) (thickness 0.1422)) (justify left bottom)))
-		(property "Footprint" "memory-v1.3-eagle:C025-025X050" (at 264.16 97.79 0) (effects (font (size 1.27 1.27)) (hide yes)))
-		(property "Datasheet" "" (at 264.16 97.79 0) (effects (font (size 1.27 1.27)) (hide yes)))
-		(pin "1")
-		(pin "2")
-		(instances (project "memory-v2.0" (path "/42231b4d-4c5f-cebb-da74-8d622a2f1dd4/36727bec-ef3f-c35c-0354-2dfce4bdbefc" (reference "C23") (unit 1))))
 	)
 	(symbol (lib_id "memory-v1.3-eagle:adafruit_C-US_025-025X050") (at 271.78 97.79 0) (unit 1)
@@
 	(wire (pts (xy 264.16 87.63) (xy 256.54 87.63)) (stroke (width 0) (type default)))
 	(wire (pts (xy 157.48 87.63) (xy 165.1 87.63)) (stroke (width 0) (type default)))
-	(wire (pts (xy 233.68 95.25) (xy 241.3 95.25)) (stroke (width 0) (type default)))
-	(wire (pts (xy 241.3 95.25) (xy 248.92 95.25)) (stroke (width 0) (type default)))
-	(wire (pts (xy 256.54 95.25) (xy 248.92 95.25)) (stroke (width 0) (type default)))
-	(wire (pts (xy 256.54 95.25) (xy 264.16 95.25)) (stroke (width 0) (type default)))
-	(wire (pts (xy 264.16 95.25) (xy 271.78 95.25)) (stroke (width 0) (type default)))
+	(wire (pts (xy 233.68 95.25) (xy 271.78 95.25)) (stroke (width 0) (type default)))
 	(wire (pts (xy 271.78 95.25) (xy 287.02 95.25)) (stroke (width 0) (type default)))
 	(wire (pts (xy 287.02 95.25) (xy 287.02 87.63)) (stroke (width 0) (type default)))
@@
 	(junction (at 264.16 87.63) (diameter 0) (color 0 0 0 0))
 	(junction (at 256.54 87.63) (diameter 0) (color 0 0 0 0))
-	(junction (at 241.3 95.25) (diameter 0) (color 0 0 0 0))
-	(junction (at 248.92 95.25) (diameter 0) (color 0 0 0 0))
-	(junction (at 256.54 95.25) (diameter 0) (color 0 0 0 0))
-	(junction (at 264.16 95.25) (diameter 0) (color 0 0 0 0))
 	(junction (at 271.78 95.25) (diameter 0) (color 0 0 0 0))
 	(junction (at 287.02 87.63) (diameter 0) (color 0 0 0 0))
@@
 	(wire (pts (xy 279.4 80.01) (xy 287.02 80.01)) (stroke (width 0) (type default)))
 	(wire (pts (xy 157.48 80.01) (xy 165.1 80.01)) (stroke (width 0) (type default)))
-	(wire (pts (xy 233.68 102.87) (xy 241.3 102.87)) (stroke (width 0) (type default)))
-	(wire (pts (xy 241.3 102.87) (xy 248.92 102.87)) (stroke (width 0) (type default)))
-	(wire (pts (xy 248.92 102.87) (xy 256.54 102.87)) (stroke (width 0) (type default)))
-	(wire (pts (xy 256.54 102.87) (xy 264.16 102.87)) (stroke (width 0) (type default)))
-	(wire (pts (xy 264.16 102.87) (xy 271.78 102.87)) (stroke (width 0) (type default)))
+	(wire (pts (xy 233.68 102.87) (xy 271.78 102.87)) (stroke (width 0) (type default)))
 	(wire (pts (xy 271.78 102.87) (xy 302.26 102.87)) (stroke (width 0) (type default)))
 	(wire (pts (xy 302.26 102.87) (xy 302.26 80.01)) (stroke (width 0) (type default)))
@@
 	(junction (at 271.78 80.01) (diameter 0) (color 0 0 0 0))
 	(junction (at 279.4 80.01) (diameter 0) (color 0 0 0 0))
-	(junction (at 241.3 102.87) (diameter 0) (color 0 0 0 0))
-	(junction (at 248.92 102.87) (diameter 0) (color 0 0 0 0))
-	(junction (at 256.54 102.87) (diameter 0) (color 0 0 0 0))
-	(junction (at 264.16 102.87) (diameter 0) (color 0 0 0 0))
 	(junction (at 271.78 102.87) (diameter 0) (color 0 0 0 0))
 	(junction (at 287.02 80.01) (diameter 0) (color 0 0 0 0))
@@
 	(label "-REG-LD-HI" (at 218.44 205.74 90) (fields_autoplaced yes) (effects (font (size 1.778 1.778)) (justify left bottom)))
 	(polyline (pts (xy 101.6 205.74) (xy 317.5 205.74)) (stroke (width 0.5) (type default) (color 0 0 132 1)))
-	(text "Memory card v2.0: IO-ADDR0-3 (C7-C10), -IO-RD (B25), -IO-WR (B26) and -RESET (C30) also feed the\nCompactFlash section on sheet 7 (I/O ports P8 = register latch, P9 = data; its own 74LS138 IC30,\nenabled by IO-ADDR3). DATA0-7 reach its data buffer IC34 and latch IC32. v1.3 used none of the I/O\nsignals: the six labels above were X1-only local labels and are global labels now." (exclude_from_sim no) (at 111.76 236.22 0) (effects (font (size 1.778 1.778) (thickness 0.254) bold) (justify left top)))
+	(text "Memory card v2.0: IO-ADDR0-3 (C7-C10), -IO-RD (B25), -IO-WR (B26) and -RESET (C30) also feed the\nCompactFlash section on sheet 7 (I/O ports P8 = register latch, P9 = data; its own 74LS138 IC30,\nenabled by IO-ADDR3). DATA0-7 reach its data buffer IC34 and latch IC32. v1.3 used none of the I/O\nsignals: the six labels above were X1-only local labels and are global labels now.\nC20-C23 (v1.3: four 100 nF with no IC beside them, in the cap row between C19 and C24) are removed\non v2.0 (Ken, 2026-09-24); every IC keeps its own 100 nF." (exclude_from_sim no) (at 111.76 236.22 0) (effects (font (size 1.778 1.778) (thickness 0.254) bold) (justify left top)))
 )

Commit message: docs(memory): plain documentation voice in the v2.0 schematic notes, order note and 1:1 prints
The JP3, removed-caps and DASP notes on sheets 1/3/7, the JLCPCB order note and the
card-cage / power-cable lines of the 1:1 prints drop the name; regenerated with build.sh
(BUILD PASS). Copper, drill and gerbers unchanged (their regeneration differed only in
date stamps and was not committed).

Co-Authored-By: Claude Opus 5.5 <noreply@anthropic.com>
Changed lines of the file:
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@@
 	(label "-REG-LD-HI" (at 218.44 205.74 90) (fields_autoplaced yes) (effects (font (size 1.778 1.778)) (justify left bottom)))
 	(polyline (pts (xy 101.6 205.74) (xy 317.5 205.74)) (stroke (width 0.5) (type default) (color 0 0 132 1)))
-	(text "Memory card v2.0: IO-ADDR0-3 (C7-C10), -IO-RD (B25), -IO-WR (B26) and -RESET (C30) also feed the\nCompactFlash section on sheet 7 (I/O ports P8 = register latch, P9 = data; its own 74LS138 IC30,\nenabled by IO-ADDR3). DATA0-7 reach its data buffer IC34 and latch IC32. v1.3 used none of the I/O\nsignals: the six labels above were X1-only local labels and are global labels now.\nC20-C23 (v1.3: four 100 nF with no IC beside them, in the cap row between C19 and C24) are removed\non v2.0 (Ken, 2026-09-24); every IC keeps its own 100 nF." (exclude_from_sim no) (at 111.76 236.22 0) (effects (font (size 1.778 1.778) (thickness 0.254) bold) (justify left top)))
+	(text "Memory card v2.0: IO-ADDR0-3 (C7-C10), -IO-RD (B25), -IO-WR (B26) and -RESET (C30) also feed the\nCompactFlash section on sheet 7 (I/O ports P8 = register latch, P9 = data; its own 74LS138 IC30,\nenabled by IO-ADDR3). DATA0-7 reach its data buffer IC34 and latch IC32. v1.3 used none of the I/O\nsignals: the six labels above were X1-only local labels and are global labels now.\nC20-C23 (v1.3: four 100 nF with no IC beside them, in the cap row between C19 and C24) are removed\non v2.0 (2026-09-24); every IC keeps its own 100 nF." (exclude_from_sim no) (at 111.76 236.22 0) (effects (font (size 1.778 1.778) (thickness 0.254) bold) (justify left top)))
 )
