File: hardware/cards/memory/kicad/v1.3/memory-v1.3-sheet3.kicad_sch (KiCad schematic)
At the start: 6 parts, among them IC1 62256P, IC10 74*00, IC13 28C64C, IC14 74*04, IC2 62256P, IC6 74*04

Commit message: fix(kicad): readable converted schematics - overlaps 42,847 -> 3,147, nothing off the frame; CF sheet 0 overlaps
- tools/kicad/sch_overlaps.py: calibrated readability check (text/text, text/body, text/line, off frame/title block)
- eagle_sch_to_kicad.py: fields placed from Eagle's smashed attributes or the symbol's >NAME/>VALUE with Eagle's align,
  size and ratio, readable angles; fields Eagle never shows hidden (FABC96R shows only its pin name); pin numbers hidden
  where every Eagle pin hides them; Eagle-hidden layers dropped (the stray SpiceOrder text); labels on their own wires,
  converter labels only where KiCad needs them; rotate-then-mirror fixed for MR90/MR270 in pin_world/no-connects;
  each sheet on the smallest page that holds it, centred clear of the title block
- finish_board.py: stable footprint-library choice (DRC counts no longer vary run to run)
- all 37 projects regenerated: netlist proofs unchanged (34 MATCH, 2 schematic-only, video Fusion export MISMATCH as
  before); DRC same or better; ERC up (loose wire ends onto graphic buses no longer hidden by labels; explained per README)
- CF card: gate names off the gate bodies, U3 clear of its title, 5.08 mm connector pins; rebuilt: DRC 0/0, proof MATCH
- schematic PDFs regenerated (tools/sch_to_pdf.py, 37/37)

Co-Authored-By: Claude Opus 5.5 <noreply@anthropic.com>
Connections:
- net MEM-RD: no longer names the net of IC6.1 (I), IC6.6 (O)
- net N$12: no longer names the net of IC10.2 (I1), IC14.10 (O)
- net N$13: no longer names the net of IC10.1 (I0), IC14.4 (O)
- net N$2: no longer names the net of IC6.3 (I), IC6.8 (O)
- net N$3: no longer names the net of IC1.22 (~{OE}), IC13.22 (~{OE}), IC2.22 (~{OE}), IC6.2 (O)
- net N$4: no longer names the net of IC1.27 (~{WE}), IC13.27 (~{WE}), IC2.27 (~{WE}), IC6.4 (O)
Other:
- note removed: "BADDR[0..15]"
- note removed: "BDATA[0..7]"
- moved on the sheet: IC1, IC13, IC2

Commit message: refactor(memory): built card is eagle/v1.3; the earlier save is eagle/deprecated/v1.3-do-not-use
Ken 2026-09-24: the memory card folders are renamed so the plain v1.3 name is the card in the machine.

- eagle/v1.3/ (earlier save, notes 2025-03-06, board 2021-03-17, NOT the built card) -> eagle/deprecated/v1.3-do-not-use/
  (git mv, contents untouched); its KiCad conversion regenerated as kicad/deprecated/v1.3-do-not-use/ (project
  memory-v1.3-do-not-use, proof MATCH 115/115, still "never fabricated").
- eagle/v1.3-fusion-export-2026-09-24/ (the BUILT card: Ken's Fusion 360 export of 2026-09-24, verified against JLCPCB
  order 2000765A) -> eagle/v1.3/; its conversion regenerated as kicad/v1.3/ (memory-v1.3.*, proof MATCH 116/116).
  verify_fab_vs_brd.py: PASS on eagle/v1.3 (all 695 holes, 1,263 tracks, parts, PnP; gerber set byte-identical to
  the one kept in the deprecated folder), FAIL on the deprecated board as before.
- Migration plan: tools/migrate_dryrun.py sends GV "Memory v1.3" to eagle/deprecated/v1.3-do-not-use/; migration/
  reports re-run (the 30 plan rows differ only by that destination). audit_tree.py: the Fusion-export rule now
  matches eagle/v1.3/ and is checked before the 2026-09-20 run log (which lists the earlier save at that path).
  Audit: 0 unexplained, 0 hash mismatches, 0 plan rows missing.
- fabricated.py -> FABRICATED.md + marker, gen_bom.py (+ docs/bom rows, --check up to date), PROVENANCE.md
  regenerated, KICAD.md rows (stale fusion-export row removed), BOARDS.md/SCHEMATICS.md rows, the memory section of
  DESIGN-REVIEW.md (now the built card: 53 parts, 169 nets, 21 ICs; the rest of that file is left at its 09-21 run).
- memory v2.0 reads ../v1.3: BASE_NAME/BASE/space_check path/docstrings/MASTER/README. The copied library is renamed
  memory-v1.3-eagle (the regenerated base's nickname; gen_mem_v2.py sch copies it with the lib tables). The converter
  derives schematic UUIDs from the project name, so in the boards a NOROUTE build does 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
Changed lines of the file:
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@@
 		(property "Intersheetrefs" "${INTERSHEET_REFS}" (at 240.03 162.56 0) (effects (font (size 1.27 1.27)) (hide yes)))
 	)
-	(label "-LO-RAM" (at 240.03 104.14 0) (fields_autoplaced yes) (effects (font (size 1.778 1.778)) (justify left bottom)))
+	(global_label "-LO-RAM" (shape passive) (at 240.03 104.14 270) (fields_autoplaced yes) (effects (font (size 1.27 1.27)) (justify right))
+		(property "Intersheetrefs" "${INTERSHEET_REFS}" (at 240.03 104.14 0) (effects (font (size 1.27 1.27)) (hide yes)))
+	)
 	(global_label "BADDR15" (shape passive) (at 95.25 109.22 180) (fields_autoplaced yes) (effects (font (size 1.27 1.27)) (justify right))
 		(property "Intersheetrefs" "${INTERSHEET_REFS}" (at 95.25 109.22 0) (effects (font (size 1.27 1.27)) (hide yes)))
