File: hardware/cards/memory/kicad/v1.3/memory-v1.3.kicad_pcb (KiCad board)
At the start: 4 copper layers, 177.8 x 114 mm, 52 parts, among them IC10 74ALS00N, IC11 74LS157N, IC12 74LS74N, IC14 74LS04N, IC18 74ALS30N, IC26 74LS374N, IC27 74LS374N, IC28 74LS374N, IC29 74LS374N, IC3 74LS32N, IC4 74ALS30N, IC5 74LS245N, IC6 74LS04N, IC7 74LS138N, IC8 74LS244N, IC9 74LS244N, X1 FABC96R

Commit message: refactor(memory): built card is eagle/v1.3; the earlier save is eagle/deprecated/v1.3-do-not-use
Ken 2026-09-24: the memory card folders are renamed so the plain v1.3 name is the card in the machine.

- eagle/v1.3/ (earlier save, notes 2025-03-06, board 2021-03-17, NOT the built card) -> eagle/deprecated/v1.3-do-not-use/
  (git mv, contents untouched); its KiCad conversion regenerated as kicad/deprecated/v1.3-do-not-use/ (project
  memory-v1.3-do-not-use, proof MATCH 115/115, still "never fabricated").
- eagle/v1.3-fusion-export-2026-09-24/ (the BUILT card: Ken's Fusion 360 export of 2026-09-24, verified against JLCPCB
  order 2000765A) -> eagle/v1.3/; its conversion regenerated as kicad/v1.3/ (memory-v1.3.*, proof MATCH 116/116).
  verify_fab_vs_brd.py: PASS on eagle/v1.3 (all 695 holes, 1,263 tracks, parts, PnP; gerber set byte-identical to
  the one kept in the deprecated folder), FAIL on the deprecated board as before.
- Migration plan: tools/migrate_dryrun.py sends GV "Memory v1.3" to eagle/deprecated/v1.3-do-not-use/; migration/
  reports re-run (the 30 plan rows differ only by that destination). audit_tree.py: the Fusion-export rule now
  matches eagle/v1.3/ and is checked before the 2026-09-20 run log (which lists the earlier save at that path).
  Audit: 0 unexplained, 0 hash mismatches, 0 plan rows missing.
- fabricated.py -> FABRICATED.md + marker, gen_bom.py (+ docs/bom rows, --check up to date), PROVENANCE.md
  regenerated, KICAD.md rows (stale fusion-export row removed), BOARDS.md/SCHEMATICS.md rows, the memory section of
  DESIGN-REVIEW.md (now the built card: 53 parts, 169 nets, 21 ICs; the rest of that file is left at its 09-21 run).
- memory v2.0 reads ../v1.3: BASE_NAME/BASE/space_check path/docstrings/MASTER/README. The copied library is renamed
  memory-v1.3-eagle (the regenerated base's nickname; gen_mem_v2.py sch copies it with the lib tables). The converter
  derives schematic UUIDs from the project name, so in the boards a NOROUTE build does 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
Parts:
- added IC15: 74ALS11N, memory-v1.3-eagle:DIL14, F.Cu at (168.9, 70.7)
- moved IC26 184.9 mm to (172.7, 18.6)
- moved IC27 184.2 mm to (172.7, 31.3)
- moved IC28 183.4 mm to (172.7, 44.0)
- moved IC29 182.5 mm to (172.7, 56.8)
- moved RN6 94.2 mm to (78.7, 115.1)
- moved RN5 75.7 mm to (50.8, 115.1)
Connections:
- net N$10 renamed RAM5
- net N$26 renamed RAM6
- net N$27 renamed RAM7
- net N$28 renamed ROM0
- net N$29 renamed ROM1
- net N$30 renamed ROM2
- net N$31 renamed ROM3
- net N$32 renamed ROM7
- net N$34 renamed ROM6
- net N$35 renamed ROM5
- net N$36 renamed SEL7
- net N$37 renamed SEL6
- net N$38 renamed SEL5
- net N$39 renamed SEL4
- net N$40 renamed SEL3
- net N$41 renamed SEL2
- net N$42 renamed SEL1
- net N$43 renamed SEL0
- net N$44 renamed ROM4
- net N$5 renamed RAM0
- net N$6 renamed RAM1
- net N$7 renamed RAM2
- net N$8 renamed RAM3
- net N$9 renamed RAM4
- IC5 pad 19: -VMA -> N$21
Routing:
- net N$33: track 0.00 -> 211.2 mm, vias 0 -> 2
- net N$47: track 0.00 -> 173.4 mm, vias 0 -> 1
- net -TMP-REG-RD1: track 0.00 -> 161.1 mm, vias 0 -> 2
- net DATA11: track 209.9 -> 365.5 mm, vias 0 -> 2
- net -TMP-REG-RD0: track 0.00 -> 155.2 mm
- net DATA7: track 156.6 -> 296.2 mm, vias 1 -> 3
- net DATA2: track 172.4 -> 303.4 mm, vias 2 -> 1
- net DATA5: track 160.6 -> 269.2 mm, vias 1 -> 4
- net DATA6: track 156.7 -> 264.6 mm, vias 1 -> 4
- net DATA3: track 174.0 -> 278.6 mm
- net DATA4: track 177.5 -> 281.7 mm, vias 2 -> 3
- net N$21: track 0.00 -> 103.3 mm
- net DATA1: track 165.6 -> 261.4 mm, vias 1 -> 5
- net DATA15: track 148.7 -> 234.9 mm
- net DATA9: track 224.3 -> 309.2 mm, vias 1 -> 2
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Other:
- board text added: "0X8000"
- board text added: "0XF000"
- board text added: "RAM"
- board text added: "ROM"
