File: hardware/cards/video/kicad/v2.0/video-v2.0-power.kicad_sch (KiCad schematic)
At the start: 58 parts, among them IC1 74ALS08, IC19 74LS00, IC20 74LS04, IC26 74LS86, IC27 7416, IC31 74LS32, IC32 74LS32, IC44 74LS74, IC45 74LS20, IC46 74LS04, IC47 74LS08, IC48 74LS10, IC53 74HCT74, IC54 74HCT08

Commit message: feat(video): V2.0 DB9 VSYNC polarity jumper JP4, board routed afresh
DB9 pin 9 now carries the 6845's VSYNC buffered by IC54/D (JP4 1-2,
+VSYNC: TV rate, IBM 5153 CGA) or inverted by IC46/F (JP4 2-3, -VSYNC:
IBM 5151 MDA); DB9 pin 2 joins pin 1 on GND. IC46/F and IC54/D were the
spare gates; IC38's fourth section is the only spare left. 121 parts,
219 nets. JP4 stands beside the DB9 with "+VS CGA" / "-VS MDA" on the silk.

The old copper could not take the change (IC46/F walled in by row A's
tracks), so build.sh routed the board from scratch: order 3 of 1, 2, 3,
7 kept, 0 unrouted, 314 vias, 22.9 m. Netlist proof MATCH 219/219, DRC 0
unconnected and no copper findings (cosmetic silk items as before),
verify PASS with 204 key connections, planes one piece each, sockets
PASS. Gerbers and zip exported again 2026-10-27; BOM, README, order
notes, BACKLOG updated; review r3 notes the board changed after it.
Not ordered.

Co-Authored-By: Claude Opus 5.5 <noreply@anthropic.com>
Parts:
- removed unit 6 of IC46
- removed unit 4 of IC54
Connections:
- no-connect marks 2 -> 0
Other:
- note added: "One 100 nF per IC beside its VCC pin (C54 at the ATmega's AVCC), C16 47 uF bulk. The bus supplies VCC and GND (X1, six pins each): the PWR_FLAGs. Spare: IC38's fourth section."
- note removed: "One 100 nF per IC beside its VCC pin (C54 at the ATmega's AVCC), C16 47 uF bulk. The bus supplies VCC and GND (X1, six pins each): the PWR_FLAGs. Spare: IC46/F (input on GND), IC54/D (inputs on GND), IC38's fourth section."
- moved on the sheet: C16, C17, C18, C19, C20, C21, C22, C23, C24, C25, C26, C27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
